Commit message: Finishing example models and adding descriptions

File: examples/3_DOF_ARM/3_DOF_ARM_description/urdf/3_DOF_ARM_description.urdf (robot description, URDF)
Before this commit: robot 3_DOF_ARM_description, 4 links, 3 joints
Links:
- link base_link: mass 0.0510508806208341 -> 0.0510508806208342
- link effector_link: mass 0.0290597320457048 -> 0.0290597320457047

File: examples/4_WHEELER/4_WHEELER_description/urdf/4_WHEELER_description.urdf (robot description, URDF)
Before this commit: robot 4_WHEELER_description, 5 links, 4 joints
Links:
- link back_right_link: mass 0.0846266521060751 -> 0.084626652106075
- link front_right_link: mass 0.084626652106075 -> 0.0846266521060751
Joints:
- joint back_left_joint: origin xyz=0.023383 0.05 -0.0099741 rpy=1.5708 0 0 -> xyz=0.0233834615384615 0.05 -0.00997411961288421 rpy=1.5707963267949 0 0
- joint back_right_joint: origin xyz=-0.051617 0.05 -0.0099741 rpy=1.5708 0 3.1416 -> xyz=-0.0516165384615385 0.05 -0.00997411961288421 rpy=1.5707963267949 0 3.14159265358979
- joint front_left_joint: origin xyz=0.023383 -0.05 -0.0099741 rpy=1.5708 0 0 -> xyz=0.0233834615384615 -0.05 -0.0099741196128842 rpy=1.5707963267949 0 0
- joint front_right_joint: origin xyz=-0.051617 -0.05 -0.0099741 rpy=1.5708 0 3.1416 -> xyz=-0.0516165384615385 -0.05 -0.00997411961288419 rpy=1.5707963267949 0 3.14159265358979

Commit message: Updating models with latest exports

File: examples/3_DOF_ARM/3_DOF_ARM_description/urdf/3_DOF_ARM_description.urdf (robot description, URDF)
Before this commit: robot 3_DOF_ARM_description, 4 links, 3 joints
Links:
- link base_link: mass 0.0510508806208342 -> 0.0510508806208341
- link effector_link: mass 0.0290597320457047 -> 0.0290597320457048
Joints:
- joint dist_joint: axis 1 0 0 -> -1 0 0; origin xyz=0 -0.18920972027972 0 rpy=-1.5707963267949 -1.78622307916987E-17 -4.68021606411955E-34 -> xyz=0 -0.18920972027972 0 rpy=-1.5707963267949 0 0
- joint effector_joint: axis 0 0 1 -> 0 0 -1; origin xyz=0 -0.18 0 rpy=1.5707963267949 7.49830360911068E-33 6.12303176911189E-17 -> xyz=0 -0.18 0 rpy=1.5707963267949 0 0
- joint prox_joint: axis 0 -1 0 -> 0 1 0; origin xyz=0.00249115384615384 0 0 rpy=-1.5707963267949 -6.12303176911189E-17 -1.5707963267949 -> xyz=0.00249115384615384 0 0 rpy=-1.5707963267949 0 -1.5707963267949

File: examples/4_WHEELER/4_WHEELER_description/urdf/4_WHEELER_description.urdf (robot description, URDF)
Before this commit: robot 4_WHEELER_description, 5 links, 4 joints
Links:
- link front_right_link: mass 0.0846266521060751 -> 0.084626652106075
Joints:
- joint back_left_joint: axis 1 0 0 -> -1 0 0
- joint back_right_joint: axis -1 0 0 -> 1 0 0
- joint front_left_joint: axis 1 0 0 -> -1 0 0
- joint front_right_joint: axis -1 0 0 -> 1 0 0
